File: KiCad Files/HUSB238_version/HUSB238_version.kicad_pcb (KiCad board)
At the start: 2 copper layers, 54 x 12.9 mm, 33 parts, among them J2 2.54_PinHeader_02x02_SMD, J3 2.54_PinHeader_02x02_SMD, J4 2.5P Terminal Block, J9 USB_C_USB2.0_14P, Q2 AONR21307, Q9 AO3400A, SW1 SW_DIP_x05, U1 LM317L_SOT-89, U3 HUSB238_USB_PD, U4 USBLC6-2SC6

Commit message: changed pcb
Parts:
- R18: value 7.8k -> 17.8k
- moved R15 6.82 mm to (149.4, 110.8)
- moved R17 6.02 mm to (163.9, 110.1), turned to 180 degrees
- moved R16 3.93 mm to (149.4, 109.5)
- moved R18 3.15 mm to (163.9, 108.7), turned to 180 degrees
Routing:
- net Net-(R16-Pad2): track 2.37 -> 0.00 mm
- net Net-(R17-Pad2): track 2.36 -> 0.00 mm
- net Net-(R15-Pad2): track 2.35 -> 0.00 mm
- net Net-(R18-Pad2): track 2.34 -> 0.00 mm
Other:
- board text added: "12V"
- board text added: "15V"
- board text added: "18V"
- board text added: "20V"
- board text added: "5V"
- board text added: "9V"
- board text added: "Down"
- board text added: "Instruction back"
- board text added: "Instructions: You can select voltages from 5-20V by putting the 1 switche up and rest down. For 20V all switches down."
- board text added: "Licensed under CC BY-NC-SA 4.0 (c) 2025 Shinui"
- board text added: "Polarity for breadboard"
- board text added: "Switches down"
- board text added: "UP"
