File: KiCad Files/CYPD3177_3.3V_V2_+_OLED/CYPD3177_3.3V_V2_+_OLED.kicad_sch (KiCad schematic)
At the start: 0 parts

Commit message: schematics done
Connections:
- no-connect marks 0 -> 3
Other:
- sheet Logic ports: added LOGIC_Report, LOGIC_SW, LOGIC_Selection, Load_Monitor_VBUS, PD_Int, PGOOD, PGOOD_Logic, RX, Rail_2, Rail_2_IN, SCL, SCL_3.3v, SDA, SDA_3.3v, TX, UPDI, VBUS_Fault, VBUS_SW; removed none
- sheet Power ports: added PD_Int, Rail_2, VBUS_Finale; removed none
- sheet Power_selection ports: added LOGIC_Report, LOGIC_SW, LOGIC_Selection, Load_Monitor_VBUS, PGOOD, PGOOD_Logic, Rail_2_IN, VBUS_Fault, VBUS_Finale, VBUS_SW; removed none

Commit message: s
Other:
- sheet Power ports: added SCL, SDA; removed none
Changed lines of the file:
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@@
+	(wire
+		(pts
+			(xy 137.16 115.57) (xy 146.05 115.57)
+		)
+		(stroke
+			(width 0)
+			(type default)
+		)
+	)
+	(wire
+		(pts
+			(xy 142.24 76.2) (xy 138.43 76.2)
+		)
+		(stroke
+			(width 0)
+			(type default)
+		)
+	)
 	(wire
 		(pts
@@
 	(wire
 		(pts
+			(xy 146.05 115.57) (xy 146.05 81.28)
+		)
+		(stroke
+			(width 0)
+			(type default)
+		)
+	)
+	(wire
+		(pts
 			(xy 152.4 120.65) (xy 152.4 102.87)
 		)
@@
 	(wire
 		(pts
+			(xy 137.16 111.76) (xy 142.24 111.76)
+		)
+		(stroke
+			(width 0)
+			(type default)
+		)
+	)
+	(wire
+		(pts
 			(xy 154.94 104.14) (xy 154.94 166.37)
 		)
@@
 	(wire
 		(pts
+			(xy 146.05 81.28) (xy 138.43 81.28)
+		)
+		(stroke
+			(width 0)
+			(type default)
+		)
+	)
+	(wire
+		(pts
 			(xy 104.14 100.33) (xy 104.14 106.68)
+		)
+		(stroke
+			(width 0)
+			(type default)
+		)
+	)
+	(wire
+		(pts
+			(xy 142.24 111.76) (xy 142.24 76.2)
 		)
 		(stroke
@@
 			(effects
 				(font
+					(size 1.27 1.27)
+				)
+				(justify right)
+			)
+		)
+		(pin "SDA" bidirectional
+			(at 138.43 81.28 0)
+			(effects
+				(font
+					(size 1.27 1.27)
+				)
+				(justify right)
+			)
+		)
+		(pin "SCL" bidirectional
+			(at 138.43 76.2 0)
+			(effects
+				(font

Commit message: changes
Other:
- title: (none) -> USB PD PPS for breadboards
Changed lines of the file:
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@@
 	(generator_version "9.0")
 	(paper "A4")
+	(title_block
+		(title "USB PD PPS for breadboards")
+		(date "2025-05-01")
+		(rev "V1")
+		(comment 1 "Licensed under CC BY-NC-SA 4.0 (c) 2025 Shinui")
+	)
 	(no_connect
 		(at 137.16 129.54)

Commit message: almost finished
Other:
- note added: "Sorry for big mess"
Changed lines of the file:
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@@
 		(comment 1 "Licensed under CC BY-NC-SA 4.0 (c) 2025 Shinui")
+	)
+	(text "Sorry for big mess"
+		(exclude_from_sim no)
+		(at 164.846 34.29 0)
+		(effects
+			(font
+				(size 1.27 1.27)
+			)
+		)
 	)
 	(no_connect
