File: KiCad Files/CYPD3177_3.3V_V2_+_OLED/Power_selection.kicad_sch (KiCad schematic)
At the start: 22 parts, among them IC1 TPS16630RGER, IC2 TPS22992SRXNR, U8 TPS2117DRL

Commit message: almost finished
Connections:
- net +5V: no longer IC1.15 (N.C_3), IC1.19 (N.C_4), IC1.20 (N.C_5), IC1.21 (N.C_6), IC1.22 (N.C_7), IC1.23 (N.C_8), IC1.24 (N.C_9), IC1.3 (N.C_1), IC1.4 (N.C_2)
- new net: IC1.15 (N.C_3), IC1.19 (N.C_4), IC1.20 (N.C_5), IC1.21 (N.C_6), IC1.22 (N.C_7), IC1.23 (N.C_8), IC1.24 (N.C_9), IC1.3 (N.C_1), IC1.4 (N.C_2)
Other:
- note added: "Selects between 5V and 3.3V for the Logic_Voltage"
- note added: "Selects between VBUS or Logic_Voltage for Rail_2_IN (which goes to shunt R)"
- moved on the sheet: C16, C18, C19, C20, R24, R25, R29, R30, R34
