File: KiCad Files/CYPD3177_3.3V_V2_+_OLED/CYPD3177_3.3V_V2_+_OLED(AFTER schotkey, BEFORE great rewring).kicad_pcb (KiCad board)
At the start: 4 copper layers, 64 x 17 mm, 94 parts, among them IC1 TPS16630RGER, IC2 TPS22992SRXNR, J1 USB_C_USB2.0_16P, J2 Conn_01x02_Pin, J3 Conn_02x05_Odd_Even, J4 Conn_02x05_Odd_Even, J5 0.91 OLED, J6 QWIIC, J7 Conn_01x05, J8 I2C_Header, Q1 DMC2990UDJ-7, SW1 GT-TC0060-H050-L1, SW2 B3U-1000P, U1 TCA9406DC, U2 INA238, U3 XC6220B331PR-G, U4 TPS62933DRLR, U5 AON7534, U6 AP33772S, U7 AON7534, U8 TPS2117DRL, U9 ATtiny3217-M

Commit message: changes
Changed lines of the file:
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@@
 		(tags "resistor")
 		(property "Reference" "R18"
-			(at 1.14 -0.008494 180)
+			(at 1.75 -0.09 180)
 			(layer "F.SilkS")
 			(effects
@@
 	)
 	(gr_line
+		(start 146.928494 82.17)
+		(end 146.718494 82.13)
+		(stroke
+			(width 0.1)
+			(type default)
+		)
+		(layer "F.SilkS")
+	)
+	(gr_line
 		(start 106.86 86.1)
 		(end 106.86 86.8)
@@
 	)
 	(gr_line
+		(start 146.928494 82.17)
+		(end 147.028494 82.04)
+		(stroke
+			(width 0.1)
+			(type default)
+		)
+		(layer "F.SilkS")
+	)
+	(gr_line
 		(start 107.21 86.45)
 		(end 106.51 86.45)
@@
 		(stroke
 			(width 0.1)
+			(type default)
+		)
+		(layer "F.SilkS")
+	)
+	(gr_line
+		(start 146.628494 81.66)
+		(end 146.928494 82.17)
+		(stroke
+			(width 0.1)
