File: KiCad Files/CYPD3177_3.3V_V2_+_OLED/CYPD3177_3.3V_V2_+_OLED(after schotly & before rewiring v2).kicad_pcb (KiCad board)
At the start: 4 copper layers, 64 x 17 mm, 94 parts, among them IC1 TPS16630RGER, IC2 TPS22992SRXNR, J1 USB_C_Receptacle_USB2.0_14P, J2 Conn_01x02_Pin, J3 Conn_02x05_Odd_Even, J4 Conn_02x05_Odd_Even, J5 0.91 OLED, J6 QWIIC, J7 Conn_01x05, J8 I2C_3.3V, Q1 DMC2990UDJ-7, SW1 GT-TC0060-H050-L1, SW2 B3U-1000P, U1 TCA9406DC, U2 INA238, U3 XC6220B331PR-G, U4 TPS62933DRLR, U5 AON7534, U6 AP33772S, U7 AON7534, U8 TPS2117DRL, U9 ATtiny3217-M

Commit message: now final version, changed routing completly and should be better board
Parts:
- C14: value 1u -> 1uF
- C19: value 1uF -> 10uF
- C23: value 100nf -> 100nF
- C24: value 22u -> 22uF
- C26: value 100uf_35V -> 100uf_35V cap
- D2: value Red Failure LED -> Failure LED
- D4: value White Status LED -> Status LED
- J1: value USB_C_Receptacle_USB2.0_14P -> USB_C_USB2.0_16P
- J8: value I2C_3.3V -> I2C_Header
- R33: value R_Shunt -> 5m; footprint Inductor_SMD:L_1206_3216Metric_Pad1.42x1.75mm_HandSolder -> Resistor_SMD:R_1206_3216Metric
- moved R25 3.77 mm to (141.1, 96.4)
- moved R34 3.76 mm to (137.7, 94.9)
- moved C23 3.57 mm to (122.2, 96.1), turned to -90 degrees
- moved R32 2.93 mm to (116.3, 93.2), turned to 180 degrees
- moved D1 1.30 mm to (112.7, 96.0)
- moved U2 1.04 mm to (118.5, 95.5)
- moved R11 0.99 mm to (114.8, 95.6), turned to 90 degrees
- moved R20 0.96 mm to (141.2, 89.2)
- moved IC2 0.74 mm to (122.0, 90.5)
- moved C21 0.74 mm to (120.5, 88.9)
- moved R30 0.74 mm to (123.6, 89.5)
- moved R31 0.74 mm to (120.4, 90.5)
- moved C22 0.48 mm to (124.0, 91.0), turned to 0 degrees
- moved C13 0.38 mm to (151.7, 94.2)
- moved R26 0.35 mm to (112.8, 94.0)
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Connections:
- C23 pad 1: +5V -> GND
- C23 pad 2: GND -> +5V
- U9 pad 1: /Logic/SW_RIGHT -> /Logic/SW_LEFT
- U9 pad 10: /Logic/SW_PRESS -> /Logic/PGOOD_Logic
- U9 pad 11: /Logic/PGOOD -> /Logic/VBUS_Fault
- U9 pad 19: /Logic/SW_LEFT -> /Logic/LOGIC_Selection
- U9 pad 2: /Logic/INA_ALERT -> /Logic/SW_RIGHT
- U9 pad 20: /Logic/LOGIC_Selection -> /Logic/LOGIC_Report
- U9 pad 21: /Logic/LOGIC_Report -> /Logic/INA_ALERT
- U9 pad 22: /Logic/SW_UP -> /Logic/LOGIC_SW
- U9 pad 24: /Logic/PGOOD_Logic -> /Logic/SW_UP
- U9 pad 7: /Logic/VBUS_Fault -> /Logic/PGOOD
- U9 pad 8: /Logic/LOGIC_SW -> /Logic/SW_PRESS
Routing:
- net /Logic/TX: track 19.8 -> 56.4 mm
- net /Logic/RX: track 21.3 -> 56.8 mm
- net Net-(D1-K): track 52.0 -> 23.9 mm, vias 4 -> 2
- net /Power/VBUS: track 19.0 -> 8.45 mm
- net /Logic/SDA_3.3v: track 26.8 -> 34.2 mm, vias 2 -> 3
- net /Power/VBUS_Finale: track 6.83 -> 13.9 mm, vias 6 -> 7
- net GND: track 115.2 -> 121.8 mm, vias 33 -> 35
- net /Logic/PGOOD_Logic: track 20.9 -> 27.3 mm, vias 2 -> 4
- net /Logic/SW_LEFT: track 43.7 -> 37.6 mm, vias 2 -> 3
- net /Logic/SW_DOWN: track 34.6 -> 40.5 mm
- net /Logic/PGOOD: track 16.7 -> 11.8 mm
- net /Logic/VBUS_Fault: track 13.8 -> 17.0 mm
- net /Logic/UPDI: track 28.3 -> 25.6 mm, vias 1 -> 2
- net /Logic/VBUS_SW: track 22.2 -> 24.3 mm, vias 2 -> 4
- net /Logic/LOGIC_Report: track 25.9 -> 28.0 mm
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- added copper zone on In1.Cu, net +5V
- added copper zone on In1.Cu, net /Logic/Rail_2
- added copper zone on In1.Cu, net /Logic/Rail_2_IN
- added copper zone on In1.Cu, net /Power/VBUS
- added copper zone on In1.Cu, net /Power/VBUS_Finale
- added copper zone on In2.Cu, net GND
- removed copper zone on In2.Cu, net +5V
- removed copper zone on In2.Cu, net /Logic/Rail_2
- removed copper zone on In2.Cu, net /Logic/Rail_2_IN
- removed copper zone on In2.Cu, net /Power/VBUS
- removed copper zone on In2.Cu, net /Power/VBUS_Finale
- removed copper zone on In1.Cu, net GND
