File: KiCad Files/CYPD3177_3.3V_V2_+_OLED/CYPD3177_3.3V_V2_+_OLED(before via changes to 0.3mm).kicad_pcb (KiCad board)
At the start: 4 copper layers, 64 x 17 mm, 93 parts, among them IC1 TPS16630RGER, IC2 TPS22992SRXNR, J1 USB_C_Receptacle_USB2.0_14P, J2 Conn_01x02_Pin, J3 Conn_02x05_Odd_Even, J4 Conn_02x05_Odd_Even, J5 0.91 OLED, J6 QWIIC, J7 Conn_01x05, J8 I2C_3.3V, Q1 2N7002DW, SW1 GT-TC0060-H050-L1, SW2 B3U-1000P, U1 TCA9406YZPR, U2 INA237, U3 XC6220B331PR-G, U4 TPS62933PDRLR, U5 AON7534, U6 AP33772S, U7 AON7534, U8 TPS2117DRL, U9 ATtiny3217-M

Commit message: changes
Parts:
- C14: value 1uF -> 1u
- D1: value Green Power LED -> Power LED
- D2: value Red Failure LED -> Failure LED
- D4: value White Status LED -> Status LED
- J1: value USB_C_Receptacle_USB2.0_14P -> USB_C_USB2.0_14P
- moved C12 0.29 mm to (135.1, 85.7)
- moved C24 0.29 mm to (137.4, 85.7)
- moved C10 0.20 mm to (139.7, 82.7)
- moved U7 0.15 mm to (140.4, 86.8)
- moved R19 0.14 mm to (144.2, 94.4)
- moved D5 0.08 mm to (131.8, 85.6)
Connections:
- U9 pad 20: /Logic/LOGIC_Report -> /Logic/LOGIC_Selection
- U9 pad 21: /Logic/LOGIC_Selection -> /Logic/LOGIC_Report
Routing:
- net +5V: track 102.1 -> 99.0 mm
- net GND: track 121.1 -> 118.1 mm, vias 39 -> 38
- net /Logic/SCL: track 61.0 -> 59.4 mm
- net /Logic/LOGIC_Selection: track 21.3 -> 22.8 mm
- net /Logic/INA_ALERT: track 33.4 -> 32.0 mm
- net /Power/USB_P: track 10.0 -> 8.75 mm
- net /Power/VBUS: track 18.7 -> 20.0 mm
- net Net-(U6-VOUT): track 8.26 -> 6.99 mm
- net /Logic/LOGIC_SW: track 16.2 -> 15.0 mm
- net /Logic/Buck_Status: track 46.4 -> 45.2 mm
- net /Logic/LOGIC_Report: track 26.9 -> 25.8 mm, vias 4 -> 2
- net Net-(Q1-G2): track 4.00 -> 2.91 mm
- net /Logic/SW_UP: track 38.1 -> 37.2 mm, vias 2 -> 4
- net /Power/USB_N: track 9.29 -> 8.43 mm
- net +3.3V: track 56.4 -> 57.2 mm
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