File: KiCad Files/CYPD3177_3.3V_V2_+_OLED/Logic.kicad_sch (KiCad schematic)
At the start: 34 parts, among them J5 0.91 OLED, J6 QWIIC, J7 Conn_01x05, J8 I2C_3.3V, Q1 2N7002DW, SW1 GT-TC0060-H050-L1, SW2 B3U-1000P, U1 TCA9406YZPR, U2 INA237, U9 ATtiny3217-M

Commit message: changes
Connections:
- net LOGIC_Report: now also U9.20 (PC3); no longer U9.21 (PC4)
- net LOGIC_Selection: now also U9.21 (PC4); no longer U9.20 (PC3)
Changed lines of the file:
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@@
+	(wire
+		(pts
+			(xy 50.8 88.138) (xy 50.8 86.36)
+		)
+		(stroke
+			(width 0)
+			(type default)
+		)
+	)
 	(wire
 		(pts
@@
 		(pts
 			(xy 172.72 60.96) (xy 172.72 53.34)
-		)
-		(stroke
-			(width 0)
-			(type default)
-		)
-	)
-	(wire
-		(pts
-			(xy 50.8 87.63) (xy 50.8 86.36)
 		)
 		(stroke
@@
 	)
 	(label "SW_UP"
-		(at 50.8 87.63 180)
+		(at 50.8 88.138 180)
 		(effects
 			(font
@@
 	(hierarchical_label "LOGIC_Selection"
 		(shape input)
-		(at 50.8 81.28 180)
+		(at 50.8 83.82 180)
 		(effects
 			(font
@@
 	(hierarchical_label "LOGIC_Report"
 		(shape input)
-		(at 50.8 83.82 180)
-		(effects
-			(font
+		(at 50.8 81.28 180)
+		(effects
+			(font
