File: KiCad Files/CYPD3177_3.3V_V2_+_OLED/Power.kicad_sch (KiCad schematic)
At the start: 38 parts, among them J1 USB_C_Receptacle_USB2.0_14P, J2 Conn_01x02_Pin, J3 Conn_02x05_Odd_Even, J4 Conn_02x05_Odd_Even, U3 XC6220B331PR-G, U4 TPS62933PDRLR, U5 AON7534, U6 AP33772S, U7 AON7534

Commit message: changes
Parts:
- C12: value 22uF -> 10uF
- C24: value 22u -> 10uF
Changed lines of the file:
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@@
 			)
 		)
-		(property "Value" "22u"
+		(property "Value" "10uF"
 			(at 155.194 32.258 0)
 			(effects
@@
 			)
 		)
-		(property "Value" "22uF"
+		(property "Value" "10uF"
 			(at 147.828 32.258 0)
 			(effects

Commit message: changes
Parts:
- C14: value 1u -> 1uF
Changed lines of the file:
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@@
 			)
 		)
-		(property "Value" "1u"
+		(property "Value" "1uF"
 			(at 157.48 64.77 0)
 			(effects
