File: KiCad Files/HUSB238_3.3V_Version/HUSB238_3.3V_Version.kicad_pcb (KiCad board)
At the start: 2 copper layers, 58 x 13.6 mm, 41 parts, among them J2 Conn_02x02_Counter_Clockwise, J3 Conn_02x02_Counter_Clockwise, J4 Conn_01x02_Pin, J9 USB_C_Receptacle_USB2.0_14P, Q2 AONR21357, Q9 AO3400A, SW1 SW_DIP_x05, U1 TPS2121, U2 NCP1117-3.3_SOT223, U3 HUSB238_USB_PD, U4 USBLC6

Commit message: changes
Parts:
- removed REF**: VQFN-24-1EP_4x4mm_P0.5mm_EP2.5x2.5mm, Package_DFN_QFN:VQFN-24-1EP_4x4mm_P0.5mm_EP2.5x2.5mm
- removed REF**: SOT-323_SC-70, Package_TO_SOT_SMD:SOT-323_SC-70
- removed REF**: WSON-8-1EP_2x2mm_P0.5mm_EP0.9x1.6mm, Package_SON:WSON-8-1EP_2x2mm_P0.5mm_EP0.9x1.6mm
- removed REF**: MSOP-10-1EP_3x3mm_P0.5mm_EP1.68x1.88mm, Package_SO:MSOP-10-1EP_3x3mm_P0.5mm_EP1.68x1.88mm
- removed REF**: HTSSOP-14-1EP_4.4x5mm_P0.65mm_EP3.4x5mm_Mask3x3.1mm, Package_SO:HTSSOP-14-1EP_4.4x5mm_P0.65mm_EP3.4x5mm_Mask3x3.1mm
