File: KiCad Files/CYPD3177_DEV_BOARD/Power_selection.kicad_sch (KiCad schematic)
At the start: 21 parts, among them IC1 TPS16630RGER, IC2 TPS22992SRXNR, U8 TPS2117DRL

Commit message: changes
Parts:
- added J15, J16, J17, J18, J19, J20: Test, Connector_PinSocket_2.54mm:PinSocket_1x01_P2.54mm_Vertical, symbol Connector_Generic:Conn_01x01
- C16, C18: footprint Capacitor_SMD:C_0603_1608Metric -> Capacitor_SMD:C_0805_2012Metric
- C19, C20, C21, C22, C8: footprint Capacitor_SMD:C_0402_1005Metric -> Capacitor_SMD:C_0805_2012Metric
- R21, R22, R23, R24, R25, R27, R28, R29, R30, R31, R4: footprint Resistor_SMD:R_0402_1005Metric -> Resistor_SMD:R_0805_2012Metric
Connections:
- net LOGIC_Report: now also J20.1 (Pin_1)
- net LOGIC_SW: now also J17.1 (Pin_1)
- net LOGIC_Selection: now also J19.1 (Pin_1)
- net PGOOD_Logic: now also J18.1 (Pin_1)
- net VBUS_Fault: now also J16.1 (Pin_1)
- net VBUS_SW: now also J15.1 (Pin_1)
