File: KiCad Files/CYPD3177_DEV_BOARD/CYPD3177_DEV_BOARD.kicad_pcb (KiCad board)
At the start: 4 copper layers, 72 x 40 mm, 92 parts, among them IC1 TPS16630RGER, IC2 TPS22992SRXNR, J1 USB_C_Receptacle_USB2.0_14P, J2 Conn_01x02_Pin, J3 Conn_02x05_Odd_Even, J4 Conn_02x05_Odd_Even, J5 0.91 OLED, J7 Conn_01x05, J8 I2C_3.3V, Q1 2N7002DW, SW1 GT-TC0060-H050-L1, SW2 B3U-1000P, U1 TCA9406YZPR, U2 INA237, U3 XC6220B331PR-G, U4 TPS62933DRLR, U5 AON7534, U6 AP33772S, U7 AON7534, U8 TPS2117DRL, U9 ATtiny3217-M

Commit message: final
Parts:
- removed C/R5: 33nF, Capacitor_SMD:C_0805_2012Metric
- removed J3, J4: Conn_02x05_Odd_Even, Connector_PinHeader_2.54mm:PinHeader_2x05_P2.54mm_Vertical_SMD
- added J10: AP33 interrupt, Connector_PinSocket_2.54mm:PinSocket_1x01_P2.54mm_Vertical, F.Cu at (164.6, 100.8)
- added J11: NTC, Connector_PinSocket_2.54mm:PinSocket_1x01_P2.54mm_Vertical, F.Cu at (169.3, 99.8)
- added J12: GND, Connector_PinSocket_2.54mm:PinSocket_1x01_P2.54mm_Vertical, F.Cu at (117.5, 94.7)
- added J13: SDA, Connector_PinSocket_2.54mm:PinSocket_1x02_P2.54mm_Vertical, F.Cu at (166.2, 104.2)
- added J14: 5V, Connector_PinSocket_2.54mm:PinSocket_1x01_P2.54mm_Vertical, F.Cu at (152.3, 76.7)
- added J15: Test, Connector_PinSocket_2.54mm:PinSocket_1x01_P2.54mm_Vertical, F.Cu at (147.5, 92.3)
- added J16: VBUS_Fault, Connector_PinSocket_2.54mm:PinSocket_1x01_P2.54mm_Vertical, F.Cu at (143.6, 98.7)
- added J17: Logic_swtich, Connector_PinSocket_2.54mm:PinSocket_1x01_P2.54mm_Vertical, F.Cu at (156.6, 91.3)
- added J18: Status for Logic selection, Connector_PinSocket_2.54mm:PinSocket_1x01_P2.54mm_Vertical, F.Cu at (135.6, 72.5)
- added J19: Logic_Selection, Connector_PinSocket_2.54mm:PinSocket_1x01_P2.54mm_Vertical, F.Cu at (152.4, 80.2)
- added J20: Logic_report, Connector_PinSocket_2.54mm:PinSocket_1x01_P2.54mm_Vertical, F.Cu at (143.5, 93.6)
- added J21: GND, Connector_PinSocket_2.54mm:PinSocket_1x01_P2.54mm_Vertical, F.Cu at (173.7, 102.2)
- added J22: Alert INA237, Connector_PinSocket_2.54mm:PinSocket_1x01_P2.54mm_Vertical, F.Cu at (115.5, 83.8)
- added J23: Buck_Status, Connector_PinSocket_2.54mm:PinSocket_1x01_P2.54mm_Vertical, F.Cu at (155.8, 79.8)
- added J6: CC1, Connector_PinSocket_2.54mm:PinSocket_1x01_P2.54mm_Vertical, F.Cu at (171.2, 96.9)
- added J9: CC2, Connector_PinSocket_2.54mm:PinSocket_1x01_P2.54mm_Vertical, F.Cu at (169.3, 90.0)
- added R34: 10k, Resistor_SMD:R_0805_2012Metric, F.Cu at (159.2, 80.0)
- C14: value 1u -> 1uF
- D1: value Green Power LED -> Power LED
- D2: value Red Failure LED -> Failure LED
- D3: value TPD4E05U06DQAR -> TPD4E05U06
- D4: value White Status LED -> Status LED
- D5: value PMEG6020ER -> PMEG6020
- J1: value USB_C_Receptacle_USB2.0_14P -> USB_C_USB2.0_14P
- L1: value 3.3u -> 3.3u power inductor
- R33: value R_Shunt -> 5mΩ
- TH1: value Thermistor_NTC_10k_0402 -> NTC
- U1: value TCA9406YZPR -> TCA9406
- U3: value XC6220B331PR-G -> XC6220B331
- U4: value TPS62933DRLR -> TPS62933PDRLR
- U8: value TPS2117DRL -> TPS2117
- U9: value ATtiny3217-M -> ATtiny3217
- moved IC1 77.8 mm to (130.0, 86.4), turned to 180 degrees
- moved IC2 77.7 mm to (136.2, 77.4), turned to 180 degrees
- moved R27 77.4 mm to (123.2, 86.1), turned to 180 degrees
- moved R31 75.7 mm to (135.7, 75.3)
- moved R23 72.3 mm to (128.3, 82.2)
- moved U8 71.8 mm to (141.2, 77.4), turned to 90 degrees
- moved J2 71.2 mm to (124.8, 72.2)
- moved C22 71.2 mm to (134.4, 80.2), turned to -90 degrees
- moved R30 70.9 mm to (136.4, 80.2), turned to -90 degrees
- moved R4 70.6 mm to (124.3, 84.2), turned to 180 degrees
- moved C17 69.7 mm to (161.9, 76.4), turned to 180 degrees
- moved R29 69.2 mm to (140.3, 74.2), turned to 90 degrees
- moved R22 67.9 mm to (131.7, 82.2)
- moved C20 67.6 mm to (138.4, 75.4), turned to -90 degrees
- moved C8 67.5 mm to (124.3, 82.2)
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Connections:
- U4 pad 7: Net-(U4-SS) -> /Logic/Buck_Status
- U9 pad 1: /Logic/SW_RIGHT -> /Logic/INA_ALERT
- U9 pad 10: /Logic/SW_PRESS -> /Logic/SW_RIGHT
- U9 pad 11: /Logic/PGOOD -> /Logic/SW_PRESS
- U9 pad 12: /Logic/Load_Monitor_VBUS -> /Logic/SW_DOWN
- U9 pad 19: /Logic/SW_LEFT -> /Logic/Buck_Status
- U9 pad 2: /Logic/INA_ALERT -> /Logic/VBUS_Fault
- U9 pad 22: /Logic/SW_UP -> /Logic/PGOOD_Logic
- U9 pad 24: /Logic/PGOOD_Logic -> /Logic/LOGIC_SW
- U9 pad 7: /Logic/VBUS_Fault -> /Logic/Load_Monitor_VBUS
- U9 pad 8: /Logic/LOGIC_SW -> /Logic/SW_UP
- U9 pad 9: /Logic/SW_DOWN -> /Logic/SW_LEFT
Routing:
- net +5V: track 0.00 -> 188.9 mm, vias 0 -> 20
- net GND: track 0.00 -> 180.9 mm, vias 0 -> 52
- net /Logic/SDA: track 0.00 -> 127.1 mm, vias 0 -> 2
- net /Logic/SCL: track 0.00 -> 122.6 mm, vias 0 -> 3
- net +3.3V: track 0.00 -> 72.9 mm, vias 0 -> 3
- net /Logic/INA_ALERT: track 0.00 -> 48.1 mm, vias 0 -> 2
- net /Logic/LOGIC_Report: track 0.00 -> 41.2 mm, vias 0 -> 2
- net /Logic/VBUS_Fault: track 0.00 -> 39.7 mm, vias 0 -> 2
- net /Logic/SW_LEFT: track 0.00 -> 36.8 mm
- net /Logic/Load_Monitor_VBUS: track 0.00 -> 36.7 mm, vias 0 -> 2
- net /Logic/SW_UP: track 0.00 -> 34.6 mm
- net /Logic/SW_DOWN: track 0.00 -> 34.1 mm
- net /Logic/PGOOD_Logic: track 0.00 -> 34.0 mm, vias 0 -> 1
- net /Logic/LOGIC_SW: track 0.00 -> 31.0 mm, vias 0 -> 1
- net /Logic/SW_PRESS: track 0.00 -> 30.7 mm
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- added copper zone on F.Cu, net +3.3V
- added copper zone on B.Cu, net +5V
- added copper zone on F.Cu, net +5V
- added copper zone on F.Cu, net /Logic/Rail_2
- added copper zone on B.Cu, net /Logic/Rail_2_IN
- added copper zone on F.Cu, net /Logic/Rail_2_IN
- added copper zone on F.Cu, net /Power/Measured_VBUS
- added copper zone on B.Cu, net /Power/VBUS
- added copper zone on F.Cu, net /Power/VBUS
- added copper zone on F.Cu, net /Power/VBUS_Finale
- added copper zone on F.Cu, net /Power_selection/Logic_Voltage
- added copper zone on B.Cu, net GND
- added copper zone on F.Cu, net GND
- added copper zone on F.Cu, net Net-(U4-SW)
- added copper zone on F.Cu, net Net-(U5-Pad5_8)
Other:
- board size 72 x 40 mm -> 66 x 40 mm
- copper layers 4 -> 2
- board text added: "3.3V"
- board text added: "5V"
- board text added: "GND"
- board text added: "RX"
- board text added: "Rail_2"
- board text added: "Reset Swtich"
- board text added: "SCL"
- board text added: "SCL_5V"
- board text added: "SDA"
- board text added: "SDA_5V"
- board text added: "TX"
- board text added: "UPDI"
- board text added: "VBUS_swtich"
