File: KiCad Files/CYPD3177_DEV_BOARD/CYPD3177_DEV_BOARD.kicad_sch (KiCad schematic)
At the start: 0 parts

Commit message: changes
Other:
- sheet Logic ports: added PGOOD; removed Buck_Status
- sheet Power ports: added none; removed Buck_Status
- sheet Power_selection ports: added PGOOD; removed none
Changed lines of the file:
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@@
+	(wire
+		(pts
+			(xy 198.12 107.95) (xy 198.12 95.25)
+		)
+		(stroke
+			(width 0)
+			(type default)
+		)
+	)
 	(wire
 		(pts
@@
 	(wire
 		(pts
+			(xy 137.16 107.95) (xy 198.12 107.95)
+		)
+		(stroke
+			(width 0)
+			(type default)
+		)
+	)
+	(wire
+		(pts
 			(xy 205.74 120.65) (xy 152.4 120.65)
 		)
@@
 	(wire
 		(pts
-			(xy 87.63 139.7) (xy 76.2 139.7)
+			(xy 198.12 95.25) (xy 205.74 95.25)
 		)
 		(stroke
@@
 	(wire
 		(pts
-			(xy 76.2 139.7) (xy 76.2 88.9)
-		)
-		(stroke
-			(width 0)
-			(type default)
-		)
-	)
-	(wire
-		(pts
 			(xy 111.76 106.68) (xy 111.76 132.08)
 		)
@@
 	(wire
 		(pts
-			(xy 76.2 88.9) (xy 81.28 88.9)
-		)
-		(stroke
-			(width 0)
-			(type default)
-		)
-	)
-	(wire
-		(pts
 			(xy 147.32 104.14) (xy 116.84 104.14)
 		)
@@
 	)
 	(sheet
-		(at 87.63 106.68)
-		(size 49.53 67.945)
+		(at 88.265 106.68)
+		(size 48.895 67.945)
 		(exclude_from_sim no)
 		(in_bom yes)
@@
 		)
 		(property "Sheetname" "Logic"
-			(at 87.63 105.9684 0)
+			(at 88.265 105.9684 0)
 			(effects
 				(font
@@
 		)
 		(property "Sheetfile" "Logic.kicad_sch"
-			(at 87.63 175.2096 0)
+			(at 88.265 175.2096 0)
 			(effects
 				(font
@@
 		)
 		(pin "SCL_3.3v" bidirectional
-			(at 87.63 150.495 180)
+			(at 88.265 150.495 180)
 			(effects
 				(font
@@
 		)
 		(pin "SDA_3.3v" bidirectional
-			(at 87.63 153.035 180)
+			(at 88.265 153.035 180)
 			(effects
 				(font
@@
 			)
 		)
-		(pin "Buck_Status" output
-			(at 87.63 139.7 180)
-			(effects
-				(font
-					(size 1.27 1.27)
-				)
-				(justify left)
+		(pin "PGOOD" output
+			(at 137.16 107.95 0)
+			(effects
+				(font
+					(size 1.27 1.27)
+				)
+				(justify right)
 			)
 		)
 		(instances
-			(project "CYPD3177_3.3V_V2_+_OLED"
+			(project "CYPD3177_DEV_BOARD"
 				(path "/a370047b-ebc6-4236-825e-9462ba7e4392"
 					(page "2")
@@
 			)
 		)
+		(pin "PGOOD" output
+			(at 205.74 95.25 180)
+			(effects
+				(font
+					(size 1.27 1.27)
+				)
+				(justify left)
+			)
+		)
 		(instances
-			(project "CYPD3177_3.3V_V2_+_OLED"
+			(project "CYPD3177_DEV_BOARD"
 				(path "/a370047b-ebc6-4236-825e-9462ba7e4392"
 					(page "4")
@@
 	)
 	(sheet
-		(at 81.28 27.94)
-		(size 57.15 67.31)
+		(at 83.185 27.94)
+		(size 55.245 67.31)
 		(exclude_from_sim no)
 		(in_bom yes)
@@
 		)
 		(property "Sheetname" "Power"
-			(at 81.28 27.2284 0)
+			(at 83.185 27.2284 0)
 			(effects
 				(font
@@
 		)
 		(property "Sheetfile" "Power.kicad_sch"
-			(at 81.28 95.8346 0)
+			(at 83.185 95.8346 0)
 			(effects
 				(font
@@
 			)
 		)
-		(pin "Buck_Status" output
-			(at 81.28 88.9 180)
-			(effects
-				(font
-					(size 1.27 1.27)
-				)
-				(justify left)
-			)
-		)
 		(instances
-			(project "CYPD3177_3.3V_V2_+_OLED"
+			(project "CYPD3177_DEV_BOARD"
 				(path "/a370047b-ebc6-4236-825e-9462ba7e4392"
 					(page "3")

Commit message: final
Other:
- sheet Logic ports: added Buck_Status; removed PGOOD
- sheet Power ports: added Buck_Status; removed none
- sheet Power_selection ports: added none; removed PGOOD
Changed lines of the file:
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@@
-	(wire
-		(pts
-			(xy 198.12 107.95) (xy 198.12 95.25)
-		)
-		(stroke
-			(width 0)
-			(type default)
-		)
-	)
 	(wire
 		(pts
@@
 	(wire
 		(pts
+			(xy 83.185 85.09) (xy 76.2 85.09)
+		)
+		(stroke
+			(width 0)
+			(type default)
+		)
+	)
+	(wire
+		(pts
 			(xy 137.16 148.59) (xy 143.51 148.59)
 		)
@@
 	(wire
 		(pts
+			(xy 76.2 85.09) (xy 76.2 137.16)
+		)
+		(stroke
+			(width 0)
+			(type default)
+		)
+	)
+	(wire
+		(pts
 			(xy 147.32 115.57) (xy 147.32 104.14)
 		)
@@
 	(wire
 		(pts
-			(xy 137.16 107.95) (xy 198.12 107.95)
-		)
-		(stroke
-			(width 0)
-			(type default)
-		)
-	)
-	(wire
-		(pts
 			(xy 205.74 120.65) (xy 152.4 120.65)
 		)
@@
 	(wire
 		(pts
-			(xy 198.12 95.25) (xy 205.74 95.25)
-		)
-		(stroke
-			(width 0)
-			(type default)
-		)
-	)
-	(wire
-		(pts
 			(xy 146.05 115.57) (xy 146.05 81.28)
 		)
@@
 		(pts
 			(xy 177.8 79.375) (xy 205.74 79.375)
+		)
+		(stroke
+			(width 0)
+			(type default)
+		)
+	)
+	(wire
+		(pts
+			(xy 76.2 137.16) (xy 88.265 137.16)
 		)
 		(stroke
@@
 			)
 		)
-		(pin "PGOOD" output
-			(at 137.16 107.95 0)
-			(effects
-				(font
-					(size 1.27 1.27)
-				)
-				(justify right)
+		(pin "Buck_Status" output
+			(at 88.265 137.16 180)
+			(effects
+				(font
+					(size 1.27 1.27)
+				)
+				(justify left)
 			)
 		)
@@
 			)
 		)
-		(pin "PGOOD" output
-			(at 205.74 95.25 180)
-			(effects
-				(font
-					(size 1.27 1.27)
-				)
-				(justify left)
-			)
-		)
 		(instances
 			(project "CYPD3177_DEV_BOARD"
@@
 			)
 		)
+		(pin "Buck_Status" output
+			(at 83.185 85.09 180)
+			(effects
+				(font
+					(size 1.27 1.27)
+				)
+				(justify left)
+			)
+		)
