File: KiCad Files/CYPD3177_DEV_BOARD/Logic.kicad_sch (KiCad schematic)
At the start: 34 parts, among them J5 0.91 OLED, J6 QWIIC, J7 Conn_01x05, J8 I2C_3.3V, Q1 2N7002DW, SW1 GT-TC0060-H050-L1, SW2 B3U-1000P, U1 TCA9406YZPR, U2 INA237, U9 ATtiny3217-M

Commit message: changes
Parts:
- removed J6: QWIIC, Connector_JST:JST_SH_SM04B-SRSS-TB_1x04-1MP_P1.00mm_Horizontal, symbol Connector_Generic:Conn_01x04
- added J21, J22: Test, Connector_PinSocket_2.54mm:PinSocket_1x01_P2.54mm_Vertical, symbol Connector_Generic:Conn_01x01
- C1, C2, C23, C3: footprint Capacitor_SMD:C_0402_1005Metric -> Capacitor_SMD:C_0805_2012Metric
- D1, D2: footprint LED_SMD:LED_0603_1608Metric_Pad1.05x0.95mm_HandSolder -> LED_SMD:LED_0805_2012Metric
- R1, R10, R11, R12, R13, R2, R26, R3, R32, R35, R36, R5, R6, R7, R8, R9: footprint Resistor_SMD:R_0402_1005Metric -> Resistor_SMD:R_0805_2012Metric
Connections:
- net INA_ALERT: now also J22.1 (Pin_1)
- net Buck_Status renamed PGOOD

Commit message: final
Parts:
- removed J21: Test, Connector_PinSocket_2.54mm:PinSocket_1x01_P2.54mm_Vertical, symbol Connector_Generic:Conn_01x01
Connections:
- net PGOOD is gone; now on net SW_PRESS: U9.11 (PB5)
- net INA_ALERT: now also U9.1 (PA2); no longer U9.2 (PA3)
- net LOGIC_SW: now also U9.24 (PA1); no longer U9.8 (PA7)
- net Load_Monitor_VBUS: now also U9.7 (PA6); no longer U9.12 (PB4)
- net PGOOD_Logic: now also U9.22 (PC5); no longer U9.24 (PA1)
- net SW_DOWN: now also U9.12 (PB4); no longer U9.9 (PB7)
- net SW_LEFT: now also U9.9 (PB7); no longer U9.19 (PC2)
- net SW_PRESS: no longer U9.10 (PB6)
- net SW_RIGHT: now also U9.10 (PB6); no longer U9.1 (PA2)
- net SW_UP: now also U9.8 (PA7); no longer U9.22 (PC5)
- net VBUS_Fault: now also U9.2 (PA3); no longer U9.7 (PA6)
- new net Buck_Status: U9.19 (PC2)
Changed lines of the file:
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@@
 	(wire
 		(pts
-			(xy 50.8 87.63) (xy 50.8 86.36)
+			(xy 100.33 147.32) (xy 110.49 147.32)
 		)
 		(stroke
@@
 	(wire
 		(pts
-			(xy 100.33 147.32) (xy 110.49 147.32)
+			(xy 130.81 162.56) (xy 142.24 162.56)
 		)
 		(stroke
@@
 	(wire
 		(pts
-			(xy 130.81 162.56) (xy 142.24 162.56)
+			(xy 81.28 50.8) (xy 83.82 50.8)
 		)
 		(stroke
@@
 	(wire
 		(pts
-			(xy 81.28 50.8) (xy 83.82 50.8)
+			(xy 212.09 101.6) (xy 222.25 101.6)
 		)
 		(stroke
@@
 	(wire
 		(pts
-			(xy 212.09 101.6) (xy 222.25 101.6)
+			(xy 110.49 66.04) (xy 110.49 68.58)
 		)
 		(stroke
@@
 	(wire
 		(pts
-			(xy 110.49 66.04) (xy 110.49 68.58)
+			(xy 81.28 69.85) (xy 81.28 68.58)
 		)
 		(stroke
@@
 	)
 	(label "SW_PRESS"
-		(at 81.28 90.17 0)
+		(at 81.28 86.36 0)
 		(effects
 			(font
@@
 	)
 	(label "SW_UP"
-		(at 50.8 87.63 180)
-		(effects
-			(font
-				(size 1.27 1.27)
-			)
-			(justify right bottom)
+		(at 81.28 69.85 0)
+		(effects
+			(font
+				(size 1.27 1.27)
+			)
+			(justify left bottom)
 		)
 	)
 	(label "SW_DOWN"
-		(at 81.28 92.71 0)
+		(at 81.28 83.82 0)
 		(effects
 			(font
@@
 	)
 	(label "INA_ALERT"
-		(at 81.28 59.69 0)
+		(at 81.28 57.15 0)
 		(effects
 			(font
@@
 	)
 	(label "SW_RIGHT"
-		(at 81.28 57.15 0)
+		(at 81.28 90.17 0)
 		(effects
 			(font
@@
 	)
 	(label "SW_LEFT"
-		(at 50.8 80.01 180)
-		(effects
-			(font
-				(size 1.27 1.27)
-			)
-			(justify right bottom)
+		(at 81.28 92.71 0)
+		(effects
+			(font
+				(size 1.27 1.27)
+			)
+			(justify left bottom)
 		)
 	)
@@
 	(hierarchical_label "LOGIC_SW"
 		(shape input)
-		(at 81.28 68.58 0)
+		(at 81.28 53.34 0)
 		(effects
 			(font
@@
 	(hierarchical_label "PGOOD_Logic"
 		(shape output)
-		(at 81.28 53.34 0)
-		(effects
-			(font
-				(size 1.27 1.27)
-			)
-			(justify left)
+		(at 50.8 86.36 180)
+		(effects
+			(font
+				(size 1.27 1.27)
+			)
+			(justify right)
 		)
 	)
@@
 		)
 	)
-	(hierarchical_label "PGOOD"
-		(shape output)
-		(at 81.28 86.36 0)
-		(effects
-			(font
-				(size 1.27 1.27)
-			)
-			(justify left)
-		)
-	)
 	(hierarchical_label "TX"
 		(shape output)
@@
 		)
 	)
+	(hierarchical_label "Buck_Status"
+		(shape output)
+		(at 50.8 78.74 180)
+		(effects
+			(font
+				(size 1.27 1.27)
+			)
+			(justify right)
+		)
+	)
 	(hierarchical_label "SDA"
 		(shape bidirectional)
@@
 	(hierarchical_label "Load_Monitor_VBUS"
 		(shape output)
-		(at 81.28 83.82 0)
+		(at 81.28 66.04 0)
 		(effects
 			(font
@@
 	(hierarchical_label "VBUS_Fault"
 		(shape output)
-		(at 81.28 66.04 0)
+		(at 81.28 58.42 0)
 		(effects
 			(font
@@
 	)
 	(symbol
-		(lib_id "Connector_Generic:Conn_01x01")
-		(at 104.14 143.51 90)
-		(unit 1)
-		(exclude_from_sim no)
-		(in_bom yes)
-		(on_board yes)
-		(dnp no)
-		(property "Reference" "J21"
-			(at 101.854 143.51 90)
-			(effects
-				(font
-					(size 1.27 1.27)
-				)
-				(justify left)
-			)
-		)
-		(property "Value" "Test"
-			(at 106.934 140.716 90)
-			(effects
-				(font
-					(size 1.27 1.27)
-				)
-				(justify left)
-			)
-		)
-		(property "Footprint" "Connector_PinSocket_2.54mm:PinSocket_1x01_P2.54mm_Vertical"
-			(at 104.14 143.51 0)
-			(effects
-				(font
-					(size 1.27 1.27)
-				)
-				(hide yes)
-			)
-		)
-		(property "Datasheet" "~"
-			(at 104.14 143.51 0)
-			(effects
-				(font
-					(size 1.27 1.27)
-				)
-				(hide yes)
-			)
-		)
-		(property "Description" "Generic connector, single row, 01x01, script generated (kicad-library-utils/schlib/autogen/connector/)"
-			(at 104.14 143.51 0)
-			(effects
-				(font
-					(size 1.27 1.27)
-				)
-				(hide yes)
-			)
-		)
-		(pin "1"
-		)
-		(instances
-			(project "CYPD3177_DEV_BOARD"
-				(path "/a370047b-ebc6-4236-825e-9462ba7e4392/bd19bb82-a076-4c57-9538-864609224ca0"
-					(reference "J21")
-					(unit 1)
-				)
-			)
-		)
-	)
-	(symbol
 		(lib_id "power:+5V")
 		(at 203.2 40.64 0)
@@
 		(dnp no)
 		(property "Reference" "R12"
-			(at 31.75 147.828 90)
-			(effects
-				(font
+			(at 31.75 147.955 90)
+			(effects
+				(font
