File: KiCad Files/CYPD3177_DEV_BOARD/Power.kicad_sch (KiCad schematic)
At the start: 38 parts, among them J1 USB_C_Receptacle_USB2.0_14P, J2 Conn_01x02_Pin, J3 Conn_02x05_Odd_Even, J4 Conn_02x05_Odd_Even, U3 XC6220B331PR-G, U4 TPS62933PDRLR, U5 AON7534, U6 AP33772S, U7 AON7534

Commit message: changes
Parts:
- removed R34: 10k, Resistor_SMD:R_0402_1005Metric, symbol Device:R
- added C/R5: 33nF, Capacitor_SMD:C_0805_2012Metric, symbol Device:C
- added J10, J11, J12, J14: Test, Connector_PinSocket_2.54mm:PinSocket_1x01_P2.54mm_Vertical, symbol Connector_Generic:Conn_01x01
- added J13: Conn_01x02, Connector_PinSocket_2.54mm:PinSocket_1x02_P2.54mm_Vertical, symbol Connector_Generic:Conn_01x02
- added J6, J9: Conn_01x01, Connector_PinSocket_2.54mm:PinSocket_1x01_P2.54mm_Vertical, symbol Connector_Generic:Conn_01x01
- C11, C13, C14, C15, C17, C25, C6: footprint Capacitor_SMD:C_0402_1005Metric -> Capacitor_SMD:C_0805_2012Metric
- C4: footprint Capacitor_SMD:C_0603_1608Metric -> Capacitor_SMD:C_0805_2012Metric
- D4: footprint LED_SMD:LED_0603_1608Metric -> LED_SMD:LED_0805_2012Metric
- R14, R15, R16, R18, R19, R20: footprint Resistor_SMD:R_0402_1005Metric -> Resistor_SMD:R_0805_2012Metric
- U4: value TPS62933PDRLR -> TPS62933DRLR
Connections:
- net +5V: now also J14.1 (Pin_1)
- net CC1: now also J6.1 (Pin_1)
- net CC2: now also J9.1 (Pin_1)
- net GND: now also C/R5.2, J12.1 (Pin_1)
- net NTC: now also J11.1 (Pin_1)
- net PD_Int: now also J10.1 (Pin_1)
- net SCL: now also J13.1 (Pin_1)
- net SDA: now also J13.2 (Pin_2)
- net Buck_Status: no longer names the net of U4.7 (SS)
- net Buck_Status: now also C/R5.1
Other:
- note added: "This component(C/R5) can either be 33nF cap for ..62933DR or a 10k Resistor for ..33PDR."

Commit message: final
Parts:
- removed C/R5: 33nF, Capacitor_SMD:C_0805_2012Metric, symbol Device:C
- removed J3, J4: Conn_02x05_Odd_Even, PinHeader_2x05_P2.54mm_Vertical_SMD, symbol Connector_Generic:Conn_02x05_Odd_Even
- added J21, J23: Test, Connector_PinSocket_2.54mm:PinSocket_1x01_P2.54mm_Vertical, symbol Connector_Generic:Conn_01x01
- added R34: 10k, Resistor_SMD:R_0805_2012Metric, symbol Device:R
- U4: value TPS62933DRLR -> TPS62933PDRLR
Connections:
- net +5V: now also R34.1
- net GND: now also J21.1 (Pin_1)
- net Buck_Status: now reaches U4.7 (Status)
- net Buck_Status: now also J23.1 (Pin_1), R34.2
Other:
- note removed: "Pin headers to plug into breaboard"
- note removed: "This component(C/R5) can either be 33nF cap for ..62933DR or a 10k Resistor for ..33PDR."
