File: KiCad Files/CYPD3177_3.3V_V2_+_OLED.kicad_pcb (KiCad board)
At the start: 4 copper layers, 64 x 17 mm, 93 parts, among them IC1 TPS16630RGER, IC2 TPS22992SRXNR, J1 USB_C_Receptacle_USB2.0_14P, J2 Conn_01x02_Pin, J3 Conn_02x05_Odd_Even, J4 Conn_02x05_Odd_Even, J5 0.91 OLED, J6 QWIIC, J7 Conn_01x05, J8 I2C_3.3V, Q1 2N7002DW, SW1 GT-TC0060-H050-L1, SW2 B3U-1000P, U1 TCA9406YZPR, U2 INA237, U3 XC6220B331PR-G, U4 TPS62933PDRLR, U5 AON7534, U6 AP33772S, U7 AON7534, U8 TPS2117DRL, U9 ATtiny3217-M

Commit message: changes
Parts:
- moved C13 0.41 mm to (151.8, 94.3)
- turned D3 to 0 degrees
Routing:
- net /Power/CC1: track 10.6 -> 4.12 mm, vias 2 -> 0
- net /Power/USB_N: track 9.29 -> 3.48 mm
- net /Power/USB_P: track 10.0 -> 4.43 mm
- net /Power/CC2: track 7.03 -> 4.77 mm
- net /Power/IFB: track 1.72 -> 0.00 mm
- net GND: track 121.1 -> 120.2 mm
